File: cartboard.kicad_pcb (KiCad board)
At the start: 2 copper layers, 138 x 62 mm, 60 parts, among them P101 CONN_01X05, P201 CONN_01X08, P202 CONN_01X08, P301 USB_OTG, P302 CONN_01X02, P401 CONN_01X02, P501 CONN_01X02, P502 CONN_01X02, P503 CONN_01X02, Q501 NTD3055L104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

Commit message: Changed the silkscreen layers and set a new release
Parts:
- added G***: LOGO, cartboard:BRADY_URL_QR, B.Cu at (207.0, 75.0)
Other:
- board text added: "Designed by Brady O'Brien in 2016"
- board text added: "http://baobrien.guru/"
