File: cartboard.kicad_pcb (KiCad board)
At the start: 2 copper layers, 138 x 62 mm, 61 parts, among them P101 CONN_01X05, P201 CONN_01X08, P202 CONN_01X08, P301 USB_OTG, P302 CONN_01X02, P401 CONN_01X02, P501 CONN_01X02, P502 CONN_01X02, P503 CONN_01X02, Q501 NTD3055L104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

Commit message: Added TAPR OHL as license
Other:
- board text added: "Licensed under the TAPR Open Hardware License (www.tapr.org/OHL) Copyright 2016, Brady O'Brien"
Changed lines of the file:
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@@
-(kicad_pcb (version 4) (host pcbnew "(2016-07-20 BZR 6990)-product")
+(kicad_pcb (version 4) (host pcbnew "(2015-11-11 BZR 6310)-product")
   (general
-    (links 0)
+    (links 152)
     (no_connects 8)
-    (area 69 38.3 222.609943 106.075001)
+    (area 69.000001 38.15 222.609943 106.075001)
     (thickness 1.6)
-    (drawings 49)
+    (drawings 50)
     (tracks 886)
     (zones 0)
@@
     (nets 84)
   )
-  (page A4)
+  (page USLetter)
+  (title_block
+    (title "Rugged PSOC Board")
+    (date 2016-09-12)
+    (rev 1)
+    (company "SIUE ARC")
+    (comment 3 "Copyright 2016, Brady O'Brien")
+    (comment 4 "Licensed under the TAPR Open Hardware License (www.tapr.org/OHL)")
+  )
   (layers
     (0 F.Cu signal)
@@
     (visible_elements FFFFFFFF)
     (pcbplotparams
-      (layerselection 0x013fc_ffffffff)
-      (usegerberextensions false)
+      (layerselection 0x013fc_80000001)
+      (usegerberextensions true)
       (excludeedgelayer true)
       (linewidth 0.100000)
@@
       (hpglpenspeed 20)
       (hpglpendiameter 15)
+      (hpglpenoverlay 2)
       (psnegative false)
       (psa4output false)
@@
       (padsonsilk false)
       (subtractmaskfromsilk false)
-      (outputformat 4)
+      (outputformat 1)
       (mirror false)
       (drillshape 0)
       (scaleselection 1)
-      (outputdirectory release-v1/))
+      (outputdirectory release-v1/gerber/))
   )
   (net 0 "")
@@
       (xy 4.445 3.175)) (layer B.SilkS) (width 0.01))
   )
+  (gr_text "Licensed under the TAPR Open Hardware License (www.tapr.org/OHL)\nCopyright 2016, Brady O'Brien" (at 216.916 46.736) (layer B.SilkS)
+    (effects (font (size 1.5 1.5) (thickness 0.3)) (justify left mirror))
+  )
   (gr_text http://baobrien.guru/ (at 209 84) (layer B.SilkS)
